Commit message: 可以手动设置小车位置了；参数优化

File: simulation/car_description/urdf/steer_base/wheel.xacro (robot description, xacro)
@@ -13,6 +13,6 @@
   <!-- Properties -->
   <xacro:property name="steer_effort" value="100.0" />
-  <xacro:property name="steer_velocity" value="50.0" />
-  <xacro:property name="steer_limit_deg" value="42.0" />
+  <xacro:property name="steer_velocity" value="100.0" />
+  <xacro:property name="steer_limit_deg" value="45.0" />
   <!-- Bicycle model front steering link (required for steer_drive_controller) -->
   <xacro:macro name="front_steer"

Commit message: 111地图加了迷宫；加了python绘图:一些细微改动

File: simulation/car_description/urdf/steer_base/wheel.xacro (robot description, xacro)
@@ -12,7 +12,8 @@
   <xacro:include filename="$(find car_description)/urdf/steer_base/inertials.xacro" />
   <!-- Properties -->
-  <xacro:property name="steer_effort" value="100.0" />
-  <xacro:property name="steer_velocity" value="100.0" />
+  <xacro:property name="steer_effort" value="1000.0" />
+  <xacro:property name="steer_velocity" value="1000.0" />
   <xacro:property name="steer_limit_deg" value="45.0" />
+  <xacro:property name="deg_to_rad" value="0.01745329251994329577" />
   <!-- Bicycle model front steering link (required for steer_drive_controller) -->
   <xacro:macro name="front_steer"
