Commit message: teb调参成功；栅格地图无损转换

File: simulation/car_description/urdf/ackermann.urdf.xacro (robot description, xacro)
@@ -123,13 +123,19 @@
       <pose>0 0 0.0 0 0 0</pose>
       <visualize>false</visualize>
-      <update_rate>400</update_rate>
+      <update_rate>40</update_rate>
       <ray>
         <scan>
           <horizontal>
-            <samples>1081</samples>
+            <samples>500</samples> <!-- Change this to 500 if gazebo keeps timing out -->
             <resolution>1</resolution>
-            <min_angle>-2.3561944902</min_angle>
-            <max_angle>2.3561944902</max_angle>
+            <min_angle>-${M_PI}</min_angle>
+            <max_angle> ${M_PI}</max_angle>
           </horizontal>
+          <!-- <vertical>
+            <samples>16</samples>
+            <resolution>2</resolution>
+            <min_angle>-${15*M_PI/180.0}</min_angle>
+            <max_angle> ${15*M_PI/180.0}</max_angle>
+          </vertical> -->
         </scan>
         <range>

File: simulation/car_description/urdf/steer_base/wheel.xacro (robot description, xacro)
@@ -14,5 +14,5 @@
   <xacro:property name="steer_effort" value="100.0" />
   <xacro:property name="steer_velocity" value="50.0" />
-  <xacro:property name="steer_limit_deg" value="45.0" />
+  <xacro:property name="steer_limit_deg" value="42.0" />
   <!-- Bicycle model front steering link (required for steer_drive_controller) -->
   <xacro:macro name="front_steer"

Commit message: update car color

File: simulation/car_description/urdf/ackermann.urdf.xacro (robot description, xacro)
@@ -54,5 +54,5 @@
         <box size="${base_length} ${base_width} ${base_height}" />
       </geometry>
-      <material name="white" />
+      <material name="gray" />
     </visual>
     <collision>
@@ -88,5 +88,5 @@
   <!-- Colour -->
   <gazebo reference="base_link">
-    <material>Gazebo/White</material>
+    <material>Gazebo/Residential</material>
   </gazebo>
   <link name="lidar">

File: simulation/car_description/urdf/steer_base/wheel.xacro (robot description, xacro)
@@ -34,5 +34,5 @@
           <cylinder radius="${steer_radius}" length="${steer_thickness}" />
         </geometry>
-        <material name="yellow" />
+        <material name="white" />
       </visual>
       <collision>
@@ -67,5 +67,5 @@
     </transmission>
     <gazebo reference="${name}_steer_link">
-      <material>Gazebo/Yellow</material>
+      <material>Gazebo/White</material>
     </gazebo>
   </xacro:macro>
@@ -92,5 +92,5 @@
           <cylinder radius="${steer_radius}" length="${steer_thickness}" />
         </geometry>
-        <material name="blue" />
+        <material name="red" />
       </visual>
       <collision>
@@ -120,5 +120,5 @@
           <cylinder radius="${wheel_radius}" length="${wheel_thickness}" />
         </geometry>
-        <material name="red" />
+        <material name="black" />
       </visual>
       <collision>
@@ -160,8 +160,8 @@
     </transmission>
     <gazebo reference="${name}_steer_link">
-      <material>Gazebo/Blue</material>
+      <material>Gazebo/Red</material>
     </gazebo>
     <gazebo reference="${name}_wheel_link">
-      <material>Gazebo/Red</material>
+      <material>Gazebo/Black</material>
     </gazebo>
   </xacro:macro>
@@ -181,5 +181,5 @@
           <cylinder radius="${wheel_radius}" length="${wheel_thickness}" />
         </geometry>
-        <material name="yellow" />
+        <material name="white" />
       </visual>
       <collision>
@@ -211,5 +211,5 @@
     </transmission>
     <gazebo reference="${name}_wheel_link">
-      <material>Gazebo/Yellow</material>
+      <material>Gazebo/White</material>
     </gazebo>
   </xacro:macro>
@@ -229,5 +229,5 @@
           <cylinder radius="${wheel_radius}" length="${wheel_thickness}" />
         </geometry>
-        <material name="yellow" />
+        <material name="white" />
       </visual>
       <collision>
@@ -249,5 +249,5 @@
     </joint>
     <gazebo reference="${name}_wheel_link">
-      <material>Gazebo/Yellow</material>
+      <material>Gazebo/White</material>
     </gazebo>
     <gazebo reference="${name}_wheel_joint">
@@ -270,5 +270,5 @@
           <cylinder radius="${wheel_radius}" length="${wheel_thickness}" />
         </geometry>
-        <material name="red" />
+        <material name="black" />
       </visual>
       <collision>
@@ -300,5 +300,5 @@
     </transmission>
     <gazebo reference="${name}_wheel_link">
-      <material>Gazebo/Red</material>
+      <material>Gazebo/Black</material>
     </gazebo>
   </xacro:macro>

Commit message: update urdf

File: simulation/car_description/urdf/ackermann.urdf.xacro (robot description, xacro)
@@ -62,27 +62,41 @@
       </geometry>
     </collision>
-    <xacro:solid_cuboid_inertial rpy="0 0 0" xyz="0 0 0" mass="${base_mass}" x="${base_length}" y="${base_width}" z="${base_height}" />
+    <xacro:solid_cuboid_inertial rpy="0 0 0" xyz="0 0 0" mass="${base_mass}" x="${base_length}"
+      y="${base_width}" z="${base_height}" />
   </link>
   <!-- Front steer and rear wheel joints required for ackermann_steering_controller -->
-  <xacro:front_steer name="front" parent="base" steer_radius="${steer_radius}" steer_thickness="${steer_thickness}"
-    steer_mass="${steer_mass}" base_length="${base_length}" base_width="${base_width}" axle_offset="${axle_offset}"
+  <xacro:front_steer name="front" parent="base" steer_radius="${steer_radius}"
+    steer_thickness="${steer_thickness}"
+    steer_mass="${steer_mass}" base_length="${base_length}" base_width="${base_width}"
+    axle_offset="${axle_offset}"
     steer_height="${wheel_radius+steer_offset}"></xacro:front_steer>
   <!-- Rear Link -->
-  <xacro:rear_wheel name="rear" parent="base" wheel_radius="${wheel_radius/4}" wheel_thickness="${wheel_thickness/2}" wheel_mass="${wheel_mass/32}">
+  <xacro:rear_wheel name="rear" parent="base" wheel_radius="${wheel_radius/4}"
+    wheel_thickness="${wheel_thickness/2}" wheel_mass="${wheel_mass/32}">
     <origin xyz="${-base_length/2+axle_offset} 0 0" rpy="${-90 * deg_to_rad} 0 0" />
   </xacro:rear_wheel>
   <!-- Steerable front wheels -->
-  <xacro:front_wheel_lr name="front_right" parent="base" reflect="-1" wheel_radius="${wheel_radius}" wheel_thickness="${wheel_thickness}"
-    wheel_mass="${wheel_mass}" steer_radius="${steer_radius}" steer_thickness="${steer_thickness}" steer_mass="${steer_mass}"
-    base_length="${base_length}" base_width="${base_width}" axle_offset="${axle_offset}" steer_height="${wheel_radius+steer_offset}"></xacro:front_wheel_lr>
-  <xacro:front_wheel_lr name="front_left" parent="base" reflect="1" wheel_radius="${wheel_radius}" wheel_thickness="${wheel_thickness}"
-    wheel_mass="${wheel_mass}" steer_radius="${steer_radius}" steer_thickness="${steer_thickness}" steer_mass="${steer_mass}"
-    base_length="${base_length}" base_width="${base_width}" axle_offset="${axle_offset}" steer_height="${wheel_radius+steer_offset}"></xacro:front_wheel_lr>
+  <xacro:front_wheel_lr name="front_right" parent="base" reflect="-1" wheel_radius="${wheel_radius}"
+    wheel_thickness="${wheel_thickness}"
+    wheel_mass="${wheel_mass}" steer_radius="${steer_radius}" steer_thickness="${steer_thickness}"
+    steer_mass="${steer_mass}"
+    base_length="${base_length}" base_width="${base_width}" axle_offset="${axle_offset}"
+    steer_height="${wheel_radius+steer_offset}"></xacro:front_wheel_lr>
+  <xacro:front_wheel_lr name="front_left" parent="base" reflect="1" wheel_radius="${wheel_radius}"
+    wheel_thickness="${wheel_thickness}"
+    wheel_mass="${wheel_mass}" steer_radius="${steer_radius}" steer_thickness="${steer_thickness}"
+    steer_mass="${steer_mass}"
+    base_length="${base_length}" base_width="${base_width}" axle_offset="${axle_offset}"
+    steer_height="${wheel_radius+steer_offset}"></xacro:front_wheel_lr>
   <!-- Rear wheels -->
-  <xacro:rear_wheel_lr name="rear_right" parent="base" wheel_radius="${wheel_radius}" wheel_thickness="${wheel_thickness}" wheel_mass="${wheel_mass}">
-    <origin xyz="${-base_length/2+axle_offset} ${-base_width/2-axle_offset} 0" rpy="${-90 * deg_to_rad} 0 0" />
+  <xacro:rear_wheel_lr name="rear_right" parent="base" wheel_radius="${wheel_radius}"
+    wheel_thickness="${wheel_thickness}" wheel_mass="${wheel_mass}">
+    <origin xyz="${-base_length/2+axle_offset} ${-base_width/2-axle_offset} 0"
+      rpy="${-90 * deg_to_rad} 0 0" />
   </xacro:rear_wheel_lr>
-  <xacro:rear_wheel_lr name="rear_left" parent="base" wheel_radius="${wheel_radius}" wheel_thickness="${wheel_thickness}" wheel_mass="${wheel_mass}">
-    <origin xyz="${-base_length/2+axle_offset} ${+base_width/2+axle_offset} 0" rpy="${-90 * deg_to_rad} 0 0" />
+  <xacro:rear_wheel_lr name="rear_left" parent="base" wheel_radius="${wheel_radius}"
+    wheel_thickness="${wheel_thickness}" wheel_mass="${wheel_mass}">
+    <origin xyz="${-base_length/2+axle_offset} ${+base_width/2+axle_offset} 0"
+      rpy="${-90 * deg_to_rad} 0 0" />
   </xacro:rear_wheel_lr>
   <!-- Colour -->

File: simulation/car_description/urdf/steer_base/wheel.xacro (robot description, xacro)
@@ -1,5 +1,6 @@
 <?xml version="1.0"?>
 <!--
-  Robot model adapted from https://github.com/CIR-KIT/steer_drive_ros/blob/kinetic-devel/steer_drive_controller/test/common/urdf/wheel.xacro
+  Robot model adapted from
+https://github.com/CIR-KIT/steer_drive_ros/blob/kinetic-devel/steer_drive_controller/test/common/urdf/wheel.xacro
   Modifications:
     <transmissions> elements have been updated and added to 'front_steer'.
@@ -108,5 +109,7 @@
       <parent link="${parent}_link" />
       <child link="${name}_steer_link" />
-      <origin xyz="${base_length/2-axle_offset} ${reflect*(base_width/2+axle_offset)} ${steer_height}" rpy="0 0 0" />
+      <origin
+        xyz="${base_length/2-axle_offset} ${reflect*(base_width/2+axle_offset)} ${steer_height}"
+        rpy="0 0 0" />
       <axis xyz="0 0 1" />
       <limit effort="${steer_effort}"
